File: Breakout.kicad_pcb (KiCad board)
At the start: 2 copper layers, 51 x 26 mm, 2 parts

Commit message: Extended circuit board
Parts:
- removed the REF** at (139.7, 88.9)
- added G***: LOGO, Custom:GBA_Logo, F.Cu at (139.7, 80.0)
- added REF**: WEEE-Logo_5.6x8mm_SilkScreen, Symbol:WEEE-Logo_5.6x8mm_SilkScreen, B.Cu at (153.5, 84.0)
- added REF**: OSHW-Logo_5.7x6mm_SilkScreen, Symbol:OSHW-Logo_5.7x6mm_SilkScreen, B.Cu at (126.9, 84.0)
- added REF**: KiCad-Logo_5mm_SilkScreen, Symbol:KiCad-Logo_5mm_SilkScreen, B.Cu at (139.7, 84.0)
- added REF**: AGB_OPEN, Custom:AGB_open, F.Cu at (139.7, 88.9)
- moved REF** 21.8 mm to (120.7, 67.7)
Routing:
- net (no net): track 342.9 -> 1039.0 mm
Other:
- board size 51 x 26 mm -> 51 x 25.5 mm
- board text added: "Rev B"
- board text removed: "Rev A"
